File: kicad/carte-controle-moteurs-dspic.kicad_pcb (KiCad board)
At the start: 4 copper layers, 142.2 x 81.3 mm, 72 parts, among them J1 PDB, J10 PWR_IN, J11 GND, J12 5V, J13 3.3V, J14 EN, J15 MOTEUR 1, J16 MOTEUR 2, J17 L1, J18 H1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

Commit message: Finalisation du typon
Parts:
- moved J6 1.27 mm to (29.2, 41.9)
- moved J8 1.27 mm to (29.2, 110.5)
- moved J7 1.27 mm to (156.2, 41.9)
- moved J9 1.27 mm to (156.2, 110.5)
Other:
- board size 142.2 x 81.3 mm -> 137.2 x 81.3 mm
- board text added: "Carte contrôle moteurs ERACL 2018 - vX.X"
Changed lines of the file:
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@@
     (links 170)
     (no_connects 0)
-    (area 6.35 24.13 165.100001 122.364501)
+    (area 20.32 29.800999 165.100001 122.364501)
     (thickness 1.6002)
-    (drawings 8)
+    (drawings 9)
     (tracks 340)
     (zones 0)
@@
     (2 Interne2 signal)
     (31 Dessous signal)
-    (32 B.Adhes user)
-    (33 F.Adhes user)
-    (34 B.Paste user)
-    (35 F.Paste user)
-    (36 B.SilkS user)
+    (32 B.Adhes user hide)
+    (33 F.Adhes user hide)
+    (34 B.Paste user hide)
+    (35 F.Paste user hide)
+    (36 B.SilkS user hide)
     (37 F.SilkS user)
     (38 B.Mask user)
     (39 F.Mask user)
-    (40 Dwgs.User user)
-    (41 Cmts.User user)
-    (42 Eco1.User user)
-    (43 Eco2.User user)
+    (40 Dwgs.User user hide)
+    (41 Cmts.User user hide)
+    (42 Eco1.User user hide)
+    (43 Eco2.User user hide)
     (44 Edge.Cuts user)
   )
@@
     (pad_to_mask_clearance 0.254)
     (aux_axis_origin 0 0)
-    (visible_elements FFFFFFFF)
+    (visible_elements FFFFF73F)
     (pcbplotparams
       (layerselection 0x00030_80000001)
@@
   )
   (module Connectors:1pin (layer Dessus)
-    (at 27.94 41.91)
+    (at 29.21 41.91)
     (descr "module 1 pin (ou trou mecanique de percage)")
     (tags DEV)
@@
   )
   (module Connectors:1pin (layer Dessus)
-    (at 157.48 41.91)
+    (at 156.21 41.91)
     (descr "module 1 pin (ou trou mecanique de percage)")
     (tags DEV)
@@
   )
   (module Connectors:1pin (layer Dessus)
-    (at 27.94 110.49)
+    (at 29.21 110.49)
     (descr "module 1 pin (ou trou mecanique de percage)")
     (tags DEV)
@@
   )
   (module Connectors:1pin (layer Dessus)
-    (at 157.48 110.49)
+    (at 156.21 110.49)
     (descr "module 1 pin (ou trou mecanique de percage)")
     (tags DEV)
@@
     )
   )
-  (gr_line (start 157.48 35.56) (end 27.94 35.56) (angle 90) (layer Edge.Cuts) (width 0.381))
-  (gr_line (start 163.83 110.49) (end 163.83 41.91) (angle 90) (layer Edge.Cuts) (width 0.381))
-  (gr_line (start 27.94 116.84) (end 157.48 116.84) (angle 90) (layer Edge.Cuts) (width 0.381))
-  (gr_line (start 21.59 41.91) (end 21.59 110.49) (angle 90) (layer Edge.Cuts) (width 0.381))
-  (gr_arc (start 27.94 41.91) (end 21.59 41.91) (angle 90) (layer Edge.Cuts) (width 0.381))
-  (gr_arc (start 157.48 41.91) (end 157.48 35.56) (angle 90) (layer Edge.Cuts) (width 0.381))
-  (gr_arc (start 27.94 110.49) (end 27.94 116.84) (angle 90) (layer Edge.Cuts) (width 0.381))
-  (gr_arc (start 157.48 110.49) (end 163.83 110.49) (angle 90) (layer Edge.Cuts) (width 0.381))
+  (gr_text "Carte contrôle moteurs ERACL 2018 - vX.X" (at 156.21 76.2 90) (layer F.SilkS)
+    (effects (font (size 2.032 1.524) (thickness 0.3048)))
+  )
+  (gr_line (start 154.94 116.84) (end 30.48 116.84) (angle 90) (layer Edge.Cuts) (width 0.381))
+  (gr_line (start 30.48 35.56) (end 154.94 35.56) (angle 90) (layer Edge.Cuts) (width 0.381))
+  (gr_line (start 161.29 110.49) (end 161.29 41.91) (angle 90) (layer Edge.Cuts) (width 0.381))
+  (gr_line (start 24.13 41.91) (end 24.13 110.49) (angle 90) (layer Edge.Cuts) (width 0.381))
+  (gr_arc (start 30.48 41.91) (end 24.13 41.91) (angle 90) (layer Edge.Cuts) (width 0.381))
+  (gr_arc (start 154.94 41.91) (end 154.94 35.56) (angle 90) (layer Edge.Cuts) (width 0.381))
+  (gr_arc (start 30.48 110.49) (end 30.48 116.84) (angle 90) (layer Edge.Cuts) (width 0.381))
+  (gr_arc (start 154.94 110.49) (end 161.29 110.49) (angle 90) (layer Edge.Cuts) (width 0.381))
   (segment (start 45.72 109.28) (end 48.32 109.28) (width 0.59944) (layer Dessous) (net 1))
   (segment (start 102.87 113.03) (end 102.87 110.49) (width 0.59944) (layer Dessous) (net 1))
@@
     (polygon
       (pts
-        (xy 165.1 118.11) (xy 20.32 118.11) (xy 20.32 34.29) (xy 165.1 34.29)
+        (xy 165.1 118.11) (xy 20.32 118.11) (xy 20.32 105.41) (xy 33.02 105.41) (xy 33.02 83.82)
+        (xy 20.32 83.82) (xy 20.32 34.29) (xy 165.1 34.29)
       )
     )
@@
     (polygon
       (pts
-        (xy 165.1 118.11) (xy 20.32 118.11) (xy 20.32 34.29) (xy 165.1 34.29)
+        (xy 165.1 118.11) (xy 20.32 118.11) (xy 20.32 105.41) (xy 33.02 105.41) (xy 33.02 83.82)
+        (xy 20.32 83.82) (xy 20.32 34.29) (xy 165.1 34.29)
       )
     )
@@
     (polygon
       (pts
-        (xy 165.1 118.11) (xy 20.32 118.11) (xy 20.32 34.29) (xy 165.1 34.29)
+        (xy 165.1 118.11) (xy 20.32 118.11) (xy 20.32 105.41) (xy 33.02 105.41) (xy 33.02 83.82)
+        (xy 20.32 83.82) (xy 20.32 34.29) (xy 165.1 34.29)
       )
     )
@@
     (polygon
       (pts
-        (xy 165.1 118.11) (xy 20.32 118.11) (xy 20.32 34.29) (xy 165.1 34.29)
+        (xy 165.1 118.11) (xy 20.32 118.11) (xy 20.32 105.41) (xy 33.02 105.41) (xy 33.02 83.82)
+        (xy 20.32 83.82) (xy 20.32 34.29) (xy 165.1 34.29)
       )
     )

Commit message: Pré-validation CAO KiCAD
Parts:
- added REF**: Heatsink_Stonecold_HS-132_32x14mm_2xFixation1.5mm, Heatsinks:Heatsink_Stonecold_HS-132_32x14mm_2xFixation1.5mm, F.Cu at (24.8, 68.6)
- D13, D14, D15, D16, D17, D18: value 3A -> 3.3V
- J15, J16, J4, J5: footprint epsa_connect:KK_2C -> Connectors_Molex:Molex_MiniFit-JR-5569-02A2_2x01x4.20mm_Angled
- J21: value ENCODEUR 1 -> ENCO. 1
- J23: value ENCODEUR 2 -> ENCO. 2
- J3: footprint Pin_Headers:Pin_Header_Angled_2x05_Pitch2.54mm -> Pin_Headers:Pin_Header_Straight_2x05_Pitch2.54mm
- J6, J7, J8, J9: footprint Connectors:1pin -> Mounting_Holes:MountingHole_3.2mm_M3_Pad
- moved J16 17.8 mm to (117.5, 128.3), turned to 180 degrees
- moved J15 16.5 mm to (93.3, 127.0), turned to 180 degrees
- moved J5 16.5 mm to (83.2, 127.0), turned to 180 degrees
- moved J4 16.5 mm to (76.2, 127.0), turned to 180 degrees
Connections:
- J10 pad 4: Net-(J10-Pad4) -> (no net)
- J3 pad 1: Net-(J3-Pad1) -> (no net)
- J3 pad 3: Net-(J3-Pad3) -> (no net)
- J6 pad 1: Net-(J6-Pad1) -> (no net)
- J7 pad 1: Net-(J7-Pad1) -> (no net)
- J8 pad 1: Net-(J8-Pad1) -> (no net)
- J9 pad 1: Net-(J9-Pad1) -> (no net)

Commit message: Mise à jour du typon avec les nouvelles empreintes
Parts:
- R1, R10, R11, R12, R2, R3, R4, R5, R6, R7, R8, R9: footprint Resistors_THT:R_Axial_DIN0204_L3.6mm_D1.6mm_P2.54mm_Vertical -> Resistors_THT:R_Axial_DIN0204_L3.6mm_D1.6mm_P7.62mm_Horizontal
- moved D10 25.7 mm to (139.7, 87.6)
- moved D11 25.7 mm to (139.7, 92.7)
- moved D6 25.7 mm to (139.7, 85.1)
- moved D7 25.7 mm to (139.7, 90.2)
- moved J4 24.2 mm to (74.9, 102.9)
- moved J5 24.1 mm to (82.5, 102.9)
- moved D12 23.3 mm to (114.3, 92.7)
- moved D5 23.3 mm to (114.3, 85.1)
- moved D8 23.3 mm to (114.3, 90.2)
- moved D9 23.3 mm to (114.3, 87.6)
- moved J16 22.9 mm to (116.8, 105.4)
- moved J15 21.6 mm to (94.0, 105.4)
- moved D3 6.35 mm to (69.8, 92.7), turned to 0 degrees
- moved D4 6.35 mm to (87.6, 96.5)
- moved C3 4.58 mm to (77.5, 86.4)
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Connections:
- J10 pad 4: (no net) -> Net-(J10-Pad4)
- J3 pad 1: (no net) -> Net-(J3-Pad1)
- J3 pad 3: (no net) -> Net-(J3-Pad3)
- J6 pad 1: (no net) -> Net-(J6-Pad1)
- J7 pad 1: (no net) -> Net-(J7-Pad1)
- J8 pad 1: (no net) -> Net-(J8-Pad1)
- J9 pad 1: (no net) -> Net-(J9-Pad1)
Routing:
- net /QEI1_CHB: track 126.5 -> 85.2 mm
- net Net-(D7-Pad1): track 110.9 -> 152.1 mm
- net Net-(D10-Pad1): track 110.4 -> 150.6 mm
- net /ALIM_PILES: track 96.0 -> 122.5 mm
- net /ENABLE: track 111.8 -> 91.1 mm
- net +3V3: track 63.1 -> 46.8 mm
- net Net-(D5-Pad2): track 122.5 -> 138.2 mm
- net Net-(D11-Pad1): track 102.8 -> 118.5 mm
- net GND: track 86.7 -> 100.6 mm
- net Net-(R12-Pad2): track 38.4 -> 47.8 mm
- net /QEI2_CHB: track 92.0 -> 82.7 mm
- net Net-(D3-Pad2): track 3.81 -> 12.3 mm
- net /QEI2_INDEX: track 73.8 -> 68.7 mm
- net /QEI2_CHA: track 81.7 -> 76.6 mm
- net Net-(D4-Pad2): track 3.81 -> 8.15 mm
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